File: final.brd (EAGLE design)
At the start: 36.8 x 36.8 mm, 14 parts, among them IC2 MICRO_ATTINY84-SSU, IC6 LGD20H

Commit message: updated
Parts:
- added R1: 10K, microbuilder:_0805MP
- added U$2: IC_REGULATOR-3.3V-0.5A, homemade-hardware:SOT23-5
- added U$3: SWITCH_TOGGLE_SPDT, homemade-hardware:SS312SAH4
- moved U$1 118.6 mm to (-7.35, -85.0)
Connections:
- removed net +3V3: R11.1, R12.1, R9.1
- removed net VDD: U$1.4
- new net N$1: U$3.2, U$6.1
- new net VBAT: U$1.4, U$2.1, U$2.3, U$3.1
- net GND: now also U$2.2
- net SCL: now also R1.2
- net VCC: now also R1.1, R11.1, R12.1, R9.1, U$2.5
Changed lines of the file:
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@@
 <layer number="27" name="tValues" color="7" fill="1" visible="yes" active="yes"/>
 <layer number="28" name="bValues" color="7" fill="1" visible="yes" active="yes"/>
-<layer number="29" name="tStop" color="7" fill="3" visible="no" active="yes"/>
-<layer number="30" name="bStop" color="7" fill="6" visible="no" active="yes"/>
-<layer number="31" name="tCream" color="7" fill="4" visible="no" active="yes"/>
-<layer number="32" name="bCream" color="7" fill="5" visible="no" active="yes"/>
-<layer number="33" name="tFinish" color="6" fill="3" visible="no" active="yes"/>
-<layer number="34" name="bFinish" color="6" fill="6" visible="no" active="yes"/>
-<layer number="35" name="tGlue" color="7" fill="4" visible="no" active="yes"/>
-<layer number="36" name="bGlue" color="7" fill="5" visible="no" active="yes"/>
-<layer number="37" name="tTest" color="7" fill="1" visible="no" active="yes"/>
-<layer number="38" name="bTest" color="7" fill="1" visible="no" active="yes"/>
+<layer number="29" name="tStop" color="7" fill="3" visible="yes" active="yes"/>
+<layer number="30" name="bStop" color="7" fill="6" visible="yes" active="yes"/>
+<layer number="31" name="tCream" color="7" fill="4" visible="yes" active="yes"/>
+<layer number="32" name="bCream" color="7" fill="5" visible="yes" active="yes"/>
+<layer number="33" name="tFinish" color="6" fill="3" visible="yes" active="yes"/>
+<layer number="34" name="bFinish" color="6" fill="6" visible="yes" active="yes"/>
+<layer number="35" name="tGlue" color="7" fill="4" visible="yes" active="yes"/>
+<layer number="36" name="bGlue" color="7" fill="5" visible="yes" active="yes"/>
+<layer number="37" name="tTest" color="7" fill="1" visible="yes" active="yes"/>
+<layer number="38" name="bTest" color="7" fill="1" visible="yes" active="yes"/>
 <layer number="39" name="tKeepout" color="4" fill="11" visible="yes" active="yes"/>
 <layer number="40" name="bKeepout" color="1" fill="11" visible="yes" active="yes"/>
@@
 <layer number="42" name="bRestrict" color="1" fill="10" visible="yes" active="yes"/>
 <layer number="43" name="vRestrict" color="2" fill="10" visible="yes" active="yes"/>
-<layer number="44" name="Drills" color="7" fill="1" visible="no" active="yes"/>
-<layer number="45" name="Holes" color="7" fill="1" visible="no" active="yes"/>
-<layer number="46" name="Milling" color="3" fill="1" visible="no" active="yes"/>
-<layer number="47" name="Measures" color="7" fill="1" visible="no" active="yes"/>
+<layer number="44" name="Drills" color="7" fill="1" visible="yes" active="yes"/>
+<layer number="45" name="Holes" color="7" fill="1" visible="yes" active="yes"/>
+<layer number="46" name="Milling" color="3" fill="1" visible="yes" active="yes"/>
+<layer number="47" name="Measures" color="7" fill="1" visible="yes" active="yes"/>
 <layer number="48" name="Document" color="7" fill="1" visible="yes" active="yes"/>
 <layer number="49" name="Reference" color="7" fill="1" visible="yes" active="yes"/>
@@
 <attribute name="VALUE" x="21.495" y="-40.485" size="1.27" layer="27"/>
 </element>
-<element name="U$1" library="SimNeoPix" package="NEOPIX_12" value="NEOPIX_12" x="20.75" y="30.3" smashed="yes"/>
+<element name="U$1" library="SimNeoPix" package="NEOPIX_12" value="NEOPIX_12" x="-7.35" y="-84.95" smashed="yes"/>
+<element name="U$2" library="homemade-hardware" package="SOT23-5" value="IC_REGULATOR-3.3V-0.5A" x="-42.85" y="-83.45" smashed="yes">
+<attribute name="NAME" x="-43.739" y="-81.291" size="0.4064" layer="25"/>
+<attribute name="PN" value="SPX3819M5-L-3-3/TR " x="-42.85" y="-83.45" size="1.778" layer="27" display="off"/>
+<attribute name="VALUE" x="-43.8025" y="-83.6405" size="0.4064" layer="27"/>
+</element>
+<element name="R1" library="microbuilder" package="_0805MP" value="10K" x="-42.45" y="-87.65" smashed="yes">
+<attribute name="NAME" x="-44.0375" y="-86.6975" size="0.8128" layer="25" ratio="18"/>
+<attribute name="VALUE" x="-44.0375" y="-88.92" size="0.4064" layer="27" ratio="10"/>
+</element>
+<element name="U$3" library="homemade-hardware" package="SS312SAH4" value="SWITCH_TOGGLE_SPDT" x="-53.4" y="-74.65" smashed="yes">
+<attribute name="HEIGHT" value="2.9" x="-53.4" y="-74.65" size="1.778" layer="27" display="off"/>
+<attribute name="PN" value="SS312SAH4" x="-53.4" y="-74.65" size="1.778" layer="27" display="off"/>
+</element>
 </elements>
 <signals>
@@
 <contactref element="C19" pad="2"/>
 <contactref element="U$7" pad="4"/>
-<via x="-27.273" y="-66.774" extent="1-16" drill="0.3937"/>
-<via x="-25.749" y="-66.774" extent="1-16" drill="0.3937"/>
 <contactref element="C25" pad="1"/>
 <contactref element="IC6" pad="8"/>
@@
 <contactref element="U$4" pad="2"/>
 <contactref element="U$1" pad="1"/>
-<wire x1="-27.273" y1="-66.774" x2="-61.35" y2="-190.2" width="0" layer="19" extent="1-1"/>
-<wire x1="-25.749" y1="-66.774" x2="-27.273" y2="-66.774" width="0" layer="19" extent="1-1"/>
-<wire x1="-38.83" y1="-48.4258" x2="-27.273" y2="-66.774" width="0" layer="19" extent="1-1"/>
-<wire x1="-3.64" y1="-57.63" x2="-25.749" y2="-66.774" width="0" layer="19" extent="1-1"/>
+<contactref element="U$2" pad="2"/>
+<wire x1="-38.83" y1="-48.4258" x2="-42.85" y2="-84.8501" width="0" layer="19" extent="1-1"/>
+<wire x1="-15.79" y1="-70.5" x2="-38.83" y2="-48.4258" width="0" layer="19" extent="1-1"/>
+<wire x1="-3.64" y1="-57.63" x2="-15.79" y2="-70.5" width="0" layer="19" extent="1-1"/>
 <wire x1="24.35" y1="-38.41" x2="-3.64" y2="-57.63" width="0" layer="19" extent="1-1"/>
 <wire x1="21.18" y1="-29.69" x2="24.35" y2="-38.41" width="0" layer="19" extent="1-1"/>
@@
 <contactref element="IC6" pad="15"/>
 <contactref element="IC6" pad="16"/>
-<wire x1="30.52" y1="-11.955" x2="-38.83" y2="-54.1342" width="0" layer="19" extent="1-1"/>
-<wire x1="31.02" y1="-11.955" x2="30.52" y2="-11.955" width="0" layer="19" extent="1-1"/>
+<contactref element="U$2" pad="5"/>
+<contactref element="R11" pad="1"/>
+<contactref element="R1" pad="1"/>
+<contactref element="R12" pad="1"/>
+<contactref element="R9" pad="1"/>
+<wire x1="-43.8" y1="-82.0499" x2="-43.466" y2="-87.65" width="0" layer="19" extent="1-1"/>
+<wire x1="-38.83" y1="-54.1342" x2="-43.8" y2="-82.0499" width="0" layer="19" extent="1-1"/>
+<wire x1="21.18" y1="-32.23" x2="-38.83" y2="-54.1342" width="0" layer="19" extent="1-1"/>
+<wire x1="23.08" y1="-29.69" x2="21.18" y2="-32.23" width="0" layer="19" extent="1-1"/>
+<wire x1="24.924" y1="-25.88" x2="23.08" y2="-29.69" width="0" layer="19" extent="1-1"/>
+<wire x1="33.88" y1="-32.23" x2="24.924" y2="-25.88" width="0" layer="19" extent="1-1"/>
+<wire x1="37.05" y1="-24.61" x2="33.88" y2="-32.23" width="0" layer="19" extent="1-1"/>
+<wire x1="31.02" y1="-11.955" x2="37.05" y2="-24.61" width="0" layer="19" extent="1-1"/>
+<wire x1="30.52" y1="-11.955" x2="31.02" y2="-11.955" width="0" layer="19" extent="1-1"/>
 <wire x1="29.795" y1="-12.18" x2="30.52" y2="-11.955" width="0" layer="19" extent="1-1"/>
-<wire x1="37.05" y1="-24.61" x2="31.02" y2="-11.955" width="0" layer="19" extent="1-1"/>
-<wire x1="23.08" y1="-29.69" x2="37.05" y2="-24.61" width="0" layer="19" extent="1-1"/>
 </signal>
 <signal name="RTS_L">
@@
 <wire x1="29.795" y1="-13.68" x2="23.08" y2="-32.23" width="0" layer="19" extent="1-1"/>
 </signal>
-<signal name="+3V3">
-<contactref element="R9" pad="1"/>
-<contactref element="R11" pad="1"/>
-<contactref element="R12" pad="1"/>
-<wire x1="24.924" y1="-25.88" x2="21.18" y2="-32.23" width="0" layer="19" extent="1-1"/>
-<wire x1="33.88" y1="-32.23" x2="24.924" y2="-25.88" width="0" layer="19" extent="1-1"/>
-</signal>
 <signal name="CS_3.3V">
 <contactref element="R11" pad="2"/>
@@
 <signal name="SCL">
 <contactref element="IC2" pad="9"/>
+<contactref element="R1" pad="2"/>
 <contactref element="IC6" pad="2"/>
+<wire x1="-32.48" y1="-48.4258" x2="-41.434" y2="-87.65" width="0" layer="19" extent="1-1"/>
 <wire x1="29.795" y1="-12.68" x2="-32.48" y2="-48.4258" width="0" layer="19" extent="1-1"/>
 </signal>
@@
 <wire x1="22.45" y1="-38.41" x2="-36.29" y2="-48.4258" width="0" layer="19" extent="1-1"/>
 </signal>
-<signal name="VDD">
-<contactref element="U$1" pad="4"/>
-</signal>
 <signal name="DIN">
 <contactref element="IC2" pad="2"/>
 <contactref element="U$1" pad="2"/>
-<wire x1="-61.25" y1="-220.1" x2="-37.56" y2="-54.1342" width="0" layer="19" extent="1-1"/>
+<wire x1="-37.56" y1="-54.1342" x2="-15.69" y2="-100.4" width="0" layer="19" extent="1-1"/>
+</signal>
+<signal name="N$1">
+<contactref element="U$6" pad="1"/>
+<contactref element="U$3" pad="2"/>
+<wire x1="-35.29" y1="-1.765" x2="-49.92" y2="-74.65" width="0" layer="19" extent="1-1"/>
+</signal>
+<signal name="VBAT">
+<contactref element="U$3" pad="1"/>
+<contactref element="U$1" pad="4"/>
+<contactref element="U$2" pad="3"/>
+<contactref element="U$2" pad="1"/>
+<wire x1="-41.9" y1="-84.8501" x2="-43.8" y2="-84.8501" width="0" layer="19" extent="1-1"/>
+<wire x1="-49.92" y1="-76.65" x2="-43.8" y2="-84.8501" width="0" layer="19" extent="1-1"/>
+<wire x1="1.46" y1="-70.5" x2="-41.9" y2="-84.8501" width="0" layer="19" extent="1-1"/>
 </signal>
 </signals>
