File: final.sch (EAGLE design)
At the start: 14 parts, among them IC2 MICRO_ATTINY84-SSU, IC6 LGD20H

Commit message: updated
Parts:
- added R1: 10K, microbuilder:RESISTOR_0805MP
- added U$2: IC_REGULATOR-3.3V-0.5A, homemade-hardware:IC_REGULATOR-3.3V-0.5A
- added U$3: SWITCH_TOGGLE_SPDT, homemade-hardware:SWITCH_TOGGLE_SPDT
Connections:
- removed net +3V3: R11.1, R12.1, R9.1
- removed net VDD: U$1.PWR
- new net N$1: U$3.COM, U$6.+
- new net VBAT: U$1.PWR, U$2.IN, U$3.A
- net GND: now also U$2.GND
- net SCL: now also R1.2
- net VCC: now also R1.1, R11.1, R12.1, R9.1, U$2.OUT
Other:
- moved on the sheet: R12
